Commit message: Implementar definicion de ilhuicamina

File: bring_up/URDF/ilhuicamina_simplified.xacro (robot description, xacro)
@@ -127,5 +127,5 @@
     </joint>
     <!--LLANTA IZQUIERDA ENMEDIO-->
-    <link name="middle_wheel">
+    <link name="middle1_link">
         <inertial>
             <mass value="${wheel_mass}"/>
@@ -148,7 +148,7 @@
         </collision>
     </link>
-    <joint name="base_to_middle_wheel" type="continuous">
-        <parent link="base_link"/>
-        <child link="middle_wheel"/>
+    <joint name="base_to_middle1_link" type="continuous">
+        <parent link="base_link"/>
+        <child link="middle1_link"/>
         <origin rpy="${PI_2} 0 0" xyz="-0.037 0.375 0"/>
         <axis rpy="0 0 0" xyz="0 0 -1"/>
@@ -220,5 +220,5 @@
     </joint>
     <!--LLANTA DERECHA ENMEDIO-->
-    <link name="middle_wheel_2">
+    <link name="middle2_link">
         <inertial>
             <mass value="${wheel_mass}"/>
@@ -241,7 +241,7 @@
         </collision>
     </link>
-    <joint name="base_to_middle_wheel_2" type="continuous">
-        <parent link="base_link"/>
-        <child link="middle_wheel_2"/>
+    <joint name="base_to_middle2_link" type="continuous">
+        <parent link="base_link"/>
+        <child link="middle2_link"/>
         <origin rpy="${PI_2} 0 0" xyz="-0.037 -0.352 0"/>
         <axis rpy="0 0 0" xyz="0 0 -1"/>
