Commit message: Cambiar nombre de los frames

File: bring_up/URDF/QT1.xacro (robot description, xacro)
@@ -3,5 +3,5 @@
     <xacro:include filename="$(find bring_up)/URDF/QT1.gazebo"/>
     <xacro:include filename="$(find bring_up)/URDF/macros.xacro"/>
-    <xacro:include filename="lidar.xacro"/>
+    <!-- <xacro:include filename="lidar.xacro"/> -->
     <xacro:property name="base_width" value="0.7038"/>
     <xacro:property name="base_depth" value="0.3019"/>
@@ -13,5 +13,5 @@
     <xacro:property name="PI_2" value="1.570796327"/>
     <xacro:property name="PI" value="3.14159265359"/>
-    <link name="chassis_link">
+    <link name="base_link">
         <pose>0 0 0 0 0 0</pose>
         <inertial>
@@ -36,5 +36,5 @@
     </link>
 <!--
-<link name="chassis_link">
+<link name="base_link">
     <pose>0 0 0 0 0 0</pose>
     <inertial>
@@ -75,6 +75,6 @@
         </visual>
     </link>
-    <joint name="chassis_to_ZED" type="fixed">
-        <parent link="chassis_link"/>
+    <joint name="base_to_ZED" type="fixed">
+        <parent link="base_link"/>
         <child link="ZED_link"/>
         <origin xyz="0.4 0.0 0.38" rpy="0 0 0"/>
@@ -109,6 +109,6 @@
         </visual>
     </link>
-    <joint name="chassis_to_barra" type="fixed">
-        <parent link="chassis_link"/>
+    <joint name="base_to_barra" type="fixed">
+        <parent link="base_link"/>
         <child link="Barra_diferencial"/>
         <origin xyz="-0.315 0 0.389" rpy="0 0 0"/>
@@ -137,6 +137,6 @@
         </visual>
     </link>
-    <joint name="chassis_to_rotula1" type="fixed">
-        <parent link="chassis_link"/>
+    <joint name="base_to_rotula1" type="fixed">
+        <parent link="base_link"/>
         <child link="rotula_1"/>
         <origin xyz="-0.381 -0.22 0.0165" rpy="0 0 0"/>
@@ -165,6 +165,6 @@
         </visual>
     </link>
-    <joint name="chassis_to_rotula2" type="fixed">
-        <parent link="chassis_link"/>
+    <joint name="base_to_rotula2" type="fixed">
+        <parent link="base_link"/>
         <child link="rotula_2"/>
         <origin xyz="-0.381 0.22 0.0165" rpy="0 0 0"/>
@@ -193,6 +193,6 @@
         </visual>
     </link>
-    <joint name="chassis_to_tubito_1" type="fixed">
-        <parent link="chassis_link"/>
+    <joint name="base_to_tubito_1" type="fixed">
+        <parent link="base_link"/>
         <child link="Tubito_1"/>
         <origin xyz="-0.035 0.3 0.3115" rpy="0 0 ${PI}"/>
@@ -221,6 +221,6 @@
         </visual>
     </link>
-    <joint name="chassis_to_tubito_2" type="fixed">
-        <parent link="chassis_link"/>
+    <joint name="base_to_tubito_2" type="fixed">
+        <parent link="base_link"/>
         <child link="Tubito_2"/>
         <origin xyz="-0.035 -0.3 0.3115" rpy="0 0 0"/>
@@ -249,5 +249,5 @@
         </visual>
     </link>
-    <joint name="chassis_to_mclovin_left" type="fixed">
+    <joint name="base_to_mclovin_left" type="fixed">
         <parent link="Tubito_1"/>
         <child link="Mclovin_left"/>
@@ -277,5 +277,5 @@
         </visual>
     </link>
-    <joint name="chassis_to_mclovin_front" type="fixed">
+    <joint name="base_to_mclovin_front" type="fixed">
         <parent link="Tubito_1"/>
         <child link="Mclovin_front"/>
@@ -305,5 +305,5 @@
         </visual>
     </link>
-    <joint name="chassis_to_mclovin_left_2" type="fixed">
+    <joint name="base_to_mclovin_left_2" type="fixed">
         <parent link="Tubito_2"/>
         <child link="Mclovin_left_2"/>
@@ -333,5 +333,5 @@
         </visual>
     </link>
-    <joint name="chassis_to_mclovin_front_2" type="fixed">
+    <joint name="base_to_mclovin_front_2" type="fixed">
         <parent link="Tubito_2"/>
         <child link="Mclovin_front_2"/>
@@ -480,6 +480,6 @@
         </collision>
     </link>
-    <joint name="chassis_to_flwheel" type="continuous">
-        <parent link="chassis_link"/>
+    <joint name="base_to_flwheel" type="continuous">
+        <parent link="base_link"/>
         <child link="flwheel_link"/>
         <origin rpy="${PI_2} 0 0" xyz="0.386 0.375 0"/>
@@ -518,5 +518,5 @@
     </link>
     <joint name="base_to_alwheel" type="continuous">
-        <parent link="chassis_link"/>
+        <parent link="base_link"/>
         <child link="blwheel_link"/>
         <origin rpy="${PI_2} 0 0" xyz="-0.45 0.375 0"/>
@@ -554,6 +554,6 @@
         </collision>
     </link>
-    <joint name="chassis_to_middle_wheel" type="continuous">
-        <parent link="chassis_link"/>
+    <joint name="base_to_middle_wheel" type="continuous">
+        <parent link="base_link"/>
         <child link="middle_wheel"/>
         <origin rpy="${PI_2} 0 0" xyz="-0.037 0.375 0"/>
@@ -591,6 +591,6 @@
         </collision>
     </link>
-    <joint name="chassis_to_frwheel" type="continuous">
-        <parent link="chassis_link"/>
+    <joint name="base_to_frwheel" type="continuous">
+        <parent link="base_link"/>
         <child link="frwheel_link"/>
         <origin rpy="${PI_2} 0 0" xyz="0.40 -0.352 0"/>
@@ -629,5 +629,5 @@
     </link>
     <joint name="base_to_arwheel" type="continuous">
-        <parent link="chassis_link"/>
+        <parent link="base_link"/>
         <child link="brwheel_link"/>
         <origin rpy="${PI_2} 0 0" xyz="-0.45 -0.352 0"/>
@@ -665,6 +665,6 @@
         </collision>
     </link>
-    <joint name="chassis_to_middle_wheel_2" type="continuous">
-        <parent link="chassis_link"/>
+    <joint name="base_to_middle_wheel_2" type="continuous">
+        <parent link="base_link"/>
         <child link="middle_wheel_2"/>
         <origin rpy="${PI_2} 0 0" xyz="-0.037 -0.352 0"/>

File: bring_up/URDF/lidar.xacro (robot description, xacro)
@@ -1,9 +1,29 @@
 <?xml version="1.0"?>
 <robot xmlns:xacro="http://www.ros.org/wiki/xacro" >
-    <xacro:arg name="gpu" default="false"/>
-    <xacro:property name="gpu" value="false" />
-    <xacro:include filename="$(find velodyne_description)/urdf/HDL-32E.urdf.xacro"/>
-    <xacro:HDL-32E parent="chassis_link" name="velodyne2" topic="/velodyne_points2" hz="10" samples="220" gpu="${gpu}">
-        <origin xyz="0.3 0 0.45" rpy="0 0 0" />
-    </xacro:HDL-32E>
+    <!-- Definimos las dimensiones del lidar-->
+    <link name="lidar_link">
+        <inertial>
+            <mass value="0.0"/>
+            <origin xyz="0 0 0" rpy="0 0 0"/>
+            <inertia ixx="0.0" ixy="0.0" ixz="0.0" iyy="0.0" iyz="0.0" izz="0.0"/>
+        </inertial>
+        <collision>
+            <geometry>
+                <cylinder radius="0.025" length="0.04"></cylinder>
+            </geometry>
+            <origin xyz="0 0 -0.02" rpy="0 0 0"/>
+        </collision>
+        <visual>
+            <geometry>
+                <cylinder radius="0.025" length="0.04"></cylinder>
+            </geometry>
+            <origin xyz="0 0 -0.02" rpy="0 0 0"/>
+        </visual>
+    </link>
+    <!-- Definimos el joint entre el lidar y la base -->
+    <joint name="base_to_lidar" type="fixed">
+        <parent link="base_link"/>
+        <child link="lidar_link"/>
+        <origin xyz="0.3 0 0.47" rpy="0 0 0"/>
+    </joint>
 </robot>

Commit message: Funciona auto nav

File: bring_up/URDF/QT1.xacro (robot description, xacro)
@@ -526,5 +526,5 @@
     </joint>
     <!--LLANTA IZQUIERDA ENMEDIO-->
-    <link name="middle_wheel">
+    <link name="middle1_link">
         <inertial>
             <mass value="${wheel_mass}"/>
@@ -554,7 +554,7 @@
         </collision>
     </link>
-    <joint name="base_to_middle_wheel" type="continuous">
-        <parent link="base_link"/>
-        <child link="middle_wheel"/>
+    <joint name="base_to_middle1_link" type="continuous">
+        <parent link="base_link"/>
+        <child link="middle1_link"/>
         <origin rpy="${PI_2} 0 0" xyz="-0.037 0.375 0"/>
         <axis rpy="0 0 0" xyz="0 0 -1"/>
@@ -637,5 +637,5 @@
     </joint>
     <!--LLANTA DERECHA ENMEDIO-->
-    <link name="middle_wheel_2">
+    <link name="middle2_link">
         <inertial>
             <mass value="${wheel_mass}"/>
@@ -665,7 +665,7 @@
         </collision>
     </link>
-    <joint name="base_to_middle_wheel_2" type="continuous">
-        <parent link="base_link"/>
-        <child link="middle_wheel_2"/>
+    <joint name="base_to_middle2_link" type="continuous">
+        <parent link="base_link"/>
+        <child link="middle2_link"/>
         <origin rpy="${PI_2} 0 0" xyz="-0.037 -0.352 0"/>
         <axis rpy="0 0 0" xyz="0 0 -1"/>
